File: SolarPanelBoards/solar-panel-side-X-minus.kicad_sch (KiCad schematic)
At the start: 54 parts, among them J1 Conn_01x06, Q1 BSS138DWQ-7, Q2 BSS138DWQ-7, U1 OPT3001DNPT, U2 DRV8830DGQR

Commit message: New X-minus board w/ magnetorquer coils and H-bridge, I2C protection circuit
Parts:
- Q1, Q2: renamed from Q?; value MBT2222ADW1T1 -> (none); footprint Package_TO_SOT_SMD:SOT-363_SC-70-6 -> (none)
- Q3: renamed from Q1; value BSS138DWQ-7 -> (none); footprint custom-footprints:BSS138DWQ-7 -> (none); symbol symbols:BSS138DWQ-7 -> sapling:BSS138DWQ-7
- Q4: renamed from Q2; value BSS138DWQ-7 -> (none); footprint custom-footprints:BSS138DWQ-7 -> (none); symbol symbols:BSS138DWQ-7 -> sapling:BSS138DWQ-7
- R3: renamed from R8; value 10K -> (none); footprint Resistor_SMD:R_0402_1005Metric -> (none)
- R4: renamed from R17; value 10K -> (none); footprint Resistor_SMD:R_0402_1005Metric -> (none)
- U2: value DRV8830DGQR -> (none); symbol xpanel-rescue:DRV8830DGQR-symbols -> sapling:symbols_DRV8830DGQR
- renumbered C4 to C3, C3 to C4, R7 to R1, R18 to R10, R1 to R13, R2 to R14, R3 to R15, R4 to R16, R10 to R17, R16 to R2, R6 to R5, R15 to R6, R5 to R7, R13 to R8
Connections:
- net GND: now also Q4.1 (S2), Q4.4 (S1); no longer Q4.1 (S2), Q4.4 (S1), U2.11 (EP)
- net SCL: now also Q1.4 (E2), Q1.6 (C1); no longer J1.5
- net SCL1_b4iso: now also J1.5, Q1.1 (E1), Q1.3 (C2)
- net SDA: now also Q2.4 (E2), Q2.6 (C1); no longer J1.4
- net SDA1_b4iso: now also J1.4, Q2.1 (E1), Q2.3 (C2)
- net at Q3.6 (D1), R1.2, R5.1: now also Q1.5 (B2)
- net at R5.2: now also Q1.2 (B1)
- net at C3.1, R10.1: now also Q4.5 (G1); no longer Q4.2 (G2)
- net at R2.2, R6.2: now also Q2.5 (B2), Q4.6 (D1); no longer Q4.3 (D2)
- net at R6.1: now also Q2.2 (B1)
- new net: Q4.2 (G2), Q4.3 (D2), R8.1
Other:
- moved on the sheet: J1
