File: SolarPanelBoards/solar-panel-side-Y-plus.kicad_sch (KiCad schematic)
At the start: 56 parts, among them J1 Conn_01x06, U1 OPT3001DNPT

Commit message: updated sch
Connections:
- net SCL: no longer J1.5
- net SCL1_b4iso: now also J1.5
- net SDA: no longer J1.4
- net SDA1_b4iso: now also J1.4
Changed lines of the file:
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@@
     )
   )
-  (global_label "SCL" (shape input) (at 167.64 125.73 0) (fields_autoplaced)
+  (global_label "SCL1_b4iso" (shape input) (at 167.64 125.73 0) (fields_autoplaced)
     (effects (font (size 1.27 1.27)) (justify left))
-    (property "Intersheet References" "${INTERSHEET_REFS}" (id 0) (at 0 0 0)
-      (effects (font (size 1.27 1.27)) hide)
+    (property "Intersheet References" "${INTERSHEET_REFS}" (id 0) (at 180.7894 125.6506 0)
+      (effects (font (size 1.27 1.27)) (justify left) hide)
     )
   )
@@
     )
   )
-  (global_label "SDA" (shape input) (at 167.64 128.27 0) (fields_autoplaced)
+  (global_label "SDA1_b4iso" (shape input) (at 167.64 128.27 0) (fields_autoplaced)
     (effects (font (size 1.27 1.27)) (justify left))
-    (property "Intersheet References" "${INTERSHEET_REFS}" (id 0) (at 0 0 0)
-      (effects (font (size 1.27 1.27)) hide)
+    (property "Intersheet References" "${INTERSHEET_REFS}" (id 0) (at 180.8499 128.1906 0)
+      (effects (font (size 1.27 1.27)) (justify left) hide)
     )
   )

Commit message: Y Plus solar panel steps 1-4
Parts:
- removed Q? (x3): MBT2222ADW1T1, Package_TO_SOT_SMD:SOT-363_SC-70-6, symbol Transistor_BJT:MBT2222ADW1T1
- added unit 1 of Q1
- added Q2: (no value), Package_TO_SOT_SMD:SOT-363_SC-70-6, symbol Transistor_BJT:MBT2222ADW1T1
- Q4: renamed from Q?; value BSS138DWQ-7 -> (none); footprint custom-footprints:BSS138DWQ-7 -> (none)
- gave numbers to parts that had none: 26
Connections:
- net +3V3: now also U1.2 (ADDR)
- net GND: now also Q4.1 (S2), Q4.4 (S1); no longer Q4.1 (S2), Q4.4 (S1)
- net SCL: now also Q1.4 (E2), Q1.6 (C1)
- net SCL1_b4iso: now also Q1.3 (C2), Q1.1 (E1)
- net SDA: now also Q2.4 (E2), Q2.6 (C1); no longer U1.2 (ADDR)
- net SDA1_b4iso: now also Q2.1 (E1), Q2.3 (C2)
- net at Q3.6 (D1), R1.2, R5.1: now also Q1.5 (B2)
- net at R6.1: now also Q2.2 (B1)
- net at R2.2, R6.2: now also Q4.6 (D1), Q2.5 (B2); no longer Q4.3 (D2)
- net at C3.1, R10.1: now also Q4.5 (G1); no longer Q4.2 (G2)
- net at R5.2: now also Q1.2 (B1)
- new net: Q4.2 (G2), Q4.3 (D2), R8.1
