File: SolarPanelBoards/solar-panel-side-X-minus.kicad_pcb (KiCad board)
At the start: 2 copper layers, 82 x 99 mm, 42 parts, among them J1 Conn_01x06, Q12 BSS138DWQ-7, Q13 BSS138DWQ-7, Q7 MBT2222ADW1T1, Q8 MBT2222ADW1T1, U1 OPT3001DNPT

Commit message: final silkscreen and stencil edits, gerbers added for final purchase
Parts:
- added G***: LOGO, LOGO, B.Cu at (153.3, 117.1)
Other:
- outline, holes or cut-outs redrawn
- net class Default removed
- board text added: "For Allison and Daniel"
