File: SolarPanelBoards/solar-panel-side-X-plus.kicad_pcb (KiCad board)
At the start: 2 copper layers, 82 x 99 mm, 42 parts, among them J1 Conn_01x06, Q12 BSS138DWQ-7, Q13 BSS138DWQ-7, Q7 MBT2222ADW1T1, Q8 MBT2222ADW1T1, U1 OPT3001DNPT

Commit message: final silkscreen and stencil edits, gerbers added for final purchase
Parts:
- added G***: LOGO, LOGO, B.Cu at (138.4, 136.0)
Other:
- net class Default removed
- board text added: "Special thanks to: Kevin Kawai, Andrea Worshill, Matt Dow, and the rest of the Celestron team So that you can see your names flying above now just as you let me see the stars Rene and Els Rutten For welcoming me into their home and teaching me life lessons beyond just the scientific Erik Petigura Who over two summers taught me the skills now engrained in this satellite"
- board text added: "To those who have helped me to this moment: Marcia Alessi, who taught me how to speak and began me on my science journey Nara Lee, who guided me through my early education Rena Heinrich, who helped me write an essay that changed my life Kelly Farland, who is the best counselor alive Eric Romin, who taught me the language of the universe Tom Marsh, who inspires all his students to breach the metap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"
- board text added: "{dblquote}Las abejas zumban, sus alas como suspiros a una sorda oreja.{dblquote} - Heather Regen"
