File: SolarPanelBoards/solar-panel-side-Y-minus.kicad_pcb (KiCad board)
At the start: 2 copper layers, 82 x 99 mm, 43 parts, among them J1 Conn_01x06, Q12 BSS138DWQ-7, Q13 BSS138DWQ-7, Q7 MBT2222ADW1T1, Q8 MBT2222ADW1T1, U1 OPT3001DNPT

Commit message: final silkscreen and stencil edits, gerbers added for final purchase
Parts:
- added G***: LOGO, LOGO, F.Cu at (126.3, 52.4)
- added G***: LOGO, LOGO, F.Cu at (146.9, 55.8)
- added G***: LOGO, LOGO, F.Cu at (146.6, 62.0)
- added G***: LOGO, LOGO, F.Cu at (167.5, 52.3)
Other:
- outline, holes or cut-outs redrawn
- net class Default removed
- board text added: "To the SSI Satellite Team Grant Regen Flynn Dreilinger Jacob Mukobi Iso Porteous Ian Chang Akasha Hayden Adrian Gamarra TaNia Donatto Connor Cremers Dev Iyer Hunter Liu Spencer Wallace Elijah Kim Langston Nashold Moritz Stephan Frances Bujah Raphael Holland Ferguson Lawton Skaling"
- board text added: "{dblquote}Thank you, Mamie{dblquote} -Iso"
- board text removed: "GPS Antenna"
