File: SolarPanelBoards/solar-panel-side-Y-plus.kicad_pcb (KiCad board)
At the start: 2 copper layers, 82 x 99 mm, 43 parts, among them J1 Conn_01x06, Q12 BSS138DWQ-7, Q13 BSS138DWQ-7, Q7 MBT2222ADW1T1, Q8 MBT2222ADW1T1, U1 OPT3001DNPT

Commit message: final silkscreen and stencil edits, gerbers added for final purchase
Parts:
- added G***: LOGO, LOGO, F.Cu at (148.5, 55.3)
Other:
- outline, holes or cut-outs redrawn
- net class Default removed
- board text added: "- Beth Ann Amos -"
- board text added: "Loooooooooooooooooooong Sat"
- board text added: "Sample return beta 0.1"
- board text added: "To Helene Chusid Regen, the first chopped liver in space and to Edith Hollerbach Amos, {dblquote}Watch your step{dblquote}"
- board text added: "To my brother and sisters, I love you all Ross Regen Clare Chang Heather Regen You can say your names are in space now :-)"
- board text added: "To my friends, Isabel Benak, Isaiah Dawid, Flynn Dreilinger, Claire Lund, Brennan Megregian, Erica Okine, Keely Fuller, Devon Holland, Joey Diaz, Lucas Pauker, Chase Small, Troy Lawrence, Lydia Villa, Julia Wortman, Allen Zhu, Johnny Rabe, Tristan Abarca, Micha Galton, Steven Trinh, Ryan Murphy, Eric Shevlet, Nathaniel Tran, Kat Johnson, Mer Cummings, Paxton Scott, Gilbert Rosal, and all those wh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"
- board text added: "To my number one source of support from day one, You're the reason I have gotten to where I am today, and without you this project would not be floating in space while you hike on the Earth below."
- board text added: "Togi Togi Togi"
- board text added: "Uncle Danny for your constant interest in the universe and Michael, Serene, and Maki Regen"
- board text added: "{dblquote}Do your best and the hell with the rest{dblquote}"
- board text removed: "GPS Antenna"
