File: SolarPanelBoards/solar-panel-side-Z-minus.kicad_pcb (KiCad board)
At the start: 2 copper layers, 97 x 97.4 mm, 41 parts, among them J1 Conn_01x06, J2 SMA Connector Male, Q12 BSS138DWQ-7, Q13 BSS138DWQ-7, Q7 MBT2222ADW1T1, Q8 MBT2222ADW1T1, U1 OPT3001DNPT, U2 HHM1589D1

Commit message: final silkscreen and stencil edits, gerbers added for final purchase
Other:
- net class Default removed
- net class RF 200 removed
- net class RF 50 removed
