File: SolarPanelBoards/solar-panel-side-Z-plus.kicad_pcb (KiCad board)
At the start: 2 copper layers, 97 x 97.4 mm, 40 parts, among them J1 Conn_01x06, J3 Conn_01x02, Q12 BSS138DWQ-7, Q13 BSS138DWQ-7, Q7 MBT2222ADW1T1, Q8 MBT2222ADW1T1, U1 OPT3001DNPT

Commit message: final silkscreen and stencil edits, gerbers added for final purchase
Other:
- net class Default removed
- board text added: "{dblquote}Why is there anything?{dblquote}"
