File: BatteryBoard/batteryboard-v01c/batteryboard.kicad_pcb (KiCad board)
At the start: 2 copper layers, 95.9 x 90.2 mm, 32 parts, among them J1 KEYSTONE-1042, J2 KEYSTONE-1042, J3 KEYSTONE-1042, J4 KEYSTONE-1042, J5 KEYSTONE-1042, J6 KEYSTONE-1042, J7 MOLEX 5023520601, J8 Screw_Terminal_01x02, Q1 IRF7458, Q2 IRF7458, Q3 MMBT2222AT, U1 R5460N233AF

Commit message: final silkscreen and stencil edits, gerbers added for final purchase
Parts:
- added Ref**: Val**, batteryboard:XYZ_cubesat-bot, B.Cu at (77.2, 89.6)
- moved Ref** 1.02 mm to (99.2, 87.8)
- moved Ref** 0.33 mm to (116.0, 67.4)
Connections:
- J7 pad 6: DigitalPinTBD -> PyCubed_PA20
Routing:
- net PyCubed_PA20: track 0.00 -> 36.3 mm, vias 0 -> 2
- net DigitalPinTBD: track 36.3 -> 0.00 mm, vias 2 -> 0
Other:
- board text added: "INSTALL BATTERIES IN ORDER! Battery Board Ver.1c.3 SSI Satellites 2022 Grant Regen"
- board text removed: "INSTALL BATTERIES IN ORDER! Battery Board Ver.1c.2 SSI Satellites 2022 Grant Regen"
